Commit message: project_to_nearest_face, virtual links

File: pyroki_retarget/unitree_description/urdf/g1_retarget/main.urdf (robot description, URDF)
Before this commit: robot g1, 41 links, 40 joints
Links:
- added link head_virtual_link, mass 0.001; visual sphere radius=0.05
- added link torso_virtual_link, mass 0.001; visual sphere radius=0.05
Joints:
- added joint head_virtual_joint: type fixed, parent torso_link, child head_virtual_link, origin xyz=0.0 0 0.23 rpy=0 0 0
- added joint torso_virtual_joint: type fixed, parent torso_link, child torso_virtual_link, origin xyz=0.0 0 0.05 rpy=0 0 0
